Commit message: compatible with the dockerfile

File: description/robot_core.xacro (robot description, xacro)
@@ -39,5 +39,5 @@
             <origin xyz="0 0 0" rpy="1.5707963267949 0 3.14" />
             <geometry>
-                <mesh filename="/home/klein/manip_ws/src/bot_manip/meshes/robot_base.stl"/>
+                <mesh filename="$(find bot_manip)/meshes/robot_base.stl"/>
             </geometry>
             <material name="blue"/>
@@ -46,5 +46,5 @@
           <origin xyz="0 0 0" rpy="1.5707963267949 0 3.14" />
             <geometry>
-                <mesh filename="/home/klein/manip_ws/src/bot_manip/meshes/robot_base.stl"/>
+                <mesh filename="$(find bot_manip)/meshes/robot_base.stl"/>
             </geometry>
         </collision>
@@ -65,5 +65,5 @@
             <origin xyz="0 0 0" rpy="1.5707963267949 0 0" />
             <geometry>
-                <mesh filename="/home/klein/manip_ws/src/bot_manip/meshes/wheel.stl"/>
+                <mesh filename="$(find bot_manip)/meshes/wheel.stl"/>
             </geometry>
             <material name="black"/>
@@ -72,5 +72,5 @@
             <origin xyz="0 0 0" rpy="1.5707963267949 0 0" />
             <geometry>
-                <mesh filename="/home/klein/manip_ws/src/bot_manip/meshes/wheel.stl"/>
+                <mesh filename="$(find bot_manip)/meshes/wheel.stl"/>
             </geometry>
         </collision>
@@ -91,5 +91,5 @@
             <origin xyz="0 0 0" rpy="1.5707963267949 0 0" />
             <geometry>
-                <mesh filename="/home/klein/manip_ws/src/bot_manip/meshes/wheel.stl"/>
+                <mesh filename="$(find bot_manip)/meshes/wheel.stl"/>
             </geometry>
             <material name="black"/>
@@ -98,5 +98,5 @@
             <origin xyz="0 0 0" rpy="1.5707963267949 0 0" />
             <geometry>
-                <mesh filename="/home/klein/manip_ws/src/bot_manip/meshes/wheel.stl"/>
+                <mesh filename="$(find bot_manip)/meshes/wheel.stl"/>
             </geometry>
         </collision>
@@ -117,5 +117,5 @@
        <origin xyz="0 0 0" rpy="1.5707963267949 0 0" />
             <geometry>
-                <mesh filename="/home/klein/manip_ws/src/bot_manip/meshes/wheel.stl"/>
+                <mesh filename="$(find bot_manip)/meshes/wheel.stl"/>
             </geometry>
         <material name="black"/>
@@ -124,5 +124,5 @@
       <origin xyz="0 0 0" rpy="1.5707963267949 0 0" />
             <geometry>
-                <mesh filename="/home/klein/manip_ws/src/bot_manip/meshes/wheel.stl"/>
+                <mesh filename="$(find bot_manip)/meshes/wheel.stl"/>
             </geometry>
     </collision>
@@ -143,5 +143,6 @@
             <origin xyz="0 0 0" rpy="1.5707963267949 0 0" />
             <geometry>
-                <mesh filename="/home/klein/manip_ws/src/bot_manip/meshes/wheel.stl"/>
+                 <!-- <mesh filename="/home/klein/manip_ws/src/bot_desc1/meshes/wheel.stl"/> -->
+                <mesh filename="$(find bot_manip)/meshes/wheel.stl"/>
             </geometry>
         <material name="black"/>
@@ -150,5 +151,5 @@
             <origin xyz="0 0 0" rpy="1.5707963267949 0 0" />
             <geometry>
-                <mesh filename="/home/klein/manip_ws/src/bot_manip/meshes/wheel.stl"/>
+                <mesh filename="$(find bot_manip)/meshes/wheel.stl"/>
             </geometry>
     </collision>

Commit message: rm the comment

File: description/robot_core.xacro (robot description, xacro)
@@ -143,5 +143,4 @@
             <origin xyz="0 0 0" rpy="1.5707963267949 0 0" />
             <geometry>
-                 <!-- <mesh filename="/home/klein/manip_ws/src/bot_desc1/meshes/wheel.stl"/> -->
                 <mesh filename="$(find bot_manip)/meshes/wheel.stl"/>
             </geometry>

Commit message: add the world

File: description/robot_core.xacro (robot description, xacro)
@@ -5,5 +5,5 @@
     <xacro:property name="chassis_width" value="0.39"/>
     <xacro:property name="chassis_height" value="0.20"/>
-    <xacro:property name="chassis_mass" value="40.0"/>
+    <xacro:property name="chassis_mass" value="20.0"/>
     <xacro:property name="wheel_radius" value="0.14"/>
     <xacro:property name="wheel_thickness" value="0.06"/>
